File: Small Display.sch (KiCad schematic (older format))
At the start: 61 parts, among them M1 ESP-07, P1 CONN_2X2, P2 MOLEX_FPC_RCPT_24POS, P3 CONN_5, Q1 PHOTO-TRANSISTOR-NPN, Q2 NTR4170N, Q3 Si1304BDL, SW1 SW-SPDT, SW2 SW_PUSH, SW3 SW_PUSH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

Commit message: Add FS files
Parts:
- C2, C4: value C -> 1uF
- R10: value R -> 200
- R15: value 3R -> 3
- R4: value R -> 470
- R6: value R -> 2k
Changed lines of the file:
@@
 P 2350 1850
 F 0 "R4" V 2430 1850 40  0000 C CNN
-F 1 "R" V 2357 1851 40  0000 C CNN
+F 1 "470" V 2357 1851 40  0000 C CNN
 F 2 "Resistors_SMD:R_0603" V 2280 1850 30  0001 C CNN
 F 3 "" H 2350 1850 30  0000 C CNN
@@
 P 3750 1400
 F 0 "R6" V 3830 1400 40  0000 C CNN
-F 1 "R" V 3757 1401 40  0000 C CNN
+F 1 "2k" V 3757 1401 40  0000 C CNN
 F 2 "Resistors_SMD:R_0603" V 3680 1400 30  0001 C CNN
 F 3 "" H 3750 1400 30  0000 C CNN
@@
 P 2450 3150
 F 0 "C2" H 2450 3250 40  0000 L CNN
-F 1 "C" H 2456 3065 40  0000 L CNN
+F 1 "1uF" H 2456 3065 40  0000 L CNN
 F 2 "Capacitors_SMD:C_0603" H 2488 3000 30  0001 C CNN
 F 3 "" H 2450 3150 60  0000 C CNN
@@
 P 8850 3850
 F 0 "R15" V 8930 3850 40  0000 C CNN
-F 1 "3R" V 8857 3851 40  0000 C CNN
+F 1 "3" V 8857 3851 40  0000 C CNN
 F 2 "Resistors_SMD:R_0603" V 8780 3850 30  0001 C CNN
 F 3 "~" H 8850 3850 30  0000 C CNN
@@
 P 5950 4500
 F 0 "C4" H 5950 4600 40  0000 L CNN
-F 1 "C" H 5956 4415 40  0000 L CNN
+F 1 "1uF" H 5956 4415 40  0000 L CNN
 F 2 "Capacitors_SMD:C_0603" H 5988 4350 30  0001 C CNN
 F 3 "" H 5950 4500 60  0000 C CNN
@@
 P 3850 2800
 F 0 "R10" V 3930 2800 40  0000 C CNN
-F 1 "R" V 3857 2801 40  0000 C CNN
+F 1 "200" V 3857 2801 40  0000 C CNN
 F 2 "Resistors_SMD:R_0603" V 3780 2800 30  0001 C CNN
 F 3 "" H 3850 2800 30  0000 C CNN
