File: displaydriver.kicad_pcb (KiCad board)
At the start: 2 copper layers, 74.6 x 38.8 mm, 107 parts, among them M1 ESP-07, P1 CONN_2X2, P2 MOLEX_FPC_RCPT_24POS, P3 CONN_5, Q1 PHOTO-TRANSISTOR-NPN, Q2 NTR4170N, Q3 Si1304BDL, SW1 SW-SPDT, SW2 SW_PUSH, SW3 SW_PUSH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

Commit message: Add FS files
Parts:
- removed VIA_STITCH: VAL**, via_stitch:VIA_STITCH
- added GND25: GND, via:VIA_0.6_0.4, F.Cu at (90.2, 45.5)
- added GND46: GND, via:VIA_0.6_0.4, F.Cu at (76.9, 75.7)
- added GND46: GND, via:VIA_0.6_0.4, F.Cu at (78.8, 75.7)
- C5: moved to F.Cu
- JP1: moved to B.Cu
- moved GND25 0.77 mm to (99.8, 54.6)
- moved C5 0.63 mm to (90.0, 44.6)
- moved JP1 0.41 mm to (96.1, 78.9), turned to 0 degrees
- moved C6 0.16 mm to (63.7, 79.1)
Routing:
- net +3.3V: track 252.1 -> 251.5 mm
Other:
- board text added: "Bluetooth E-Paper Display"
- board text added: "Bluetooth E-Paper Display Zoetrope Labs 2015"
- board text added: "Bluetooth E-Paper Display Zoetrope Labs | V0.1 2015"
- board text added: "V0.1"
- board text added: "Zoetrope Labs"
